Commit message: Fixing some bugs in the canbus_init.sh in xacro and launch file. there still a problem with hardware canbus

File: omniman_ros2_control/description/nxp_omniman.urdf.xacro (robot description, xacro)
@@ -8,11 +8,8 @@
     <!-- Launch arguments -->
     <xacro:arg name="use_sim" default="false"/>
-    <xacro:arg name="canbus_base" default="can0"/>
-    <xacro:arg name="canbus_arm" default="can1"/>
-    <xacro:arg name="serial_port" default="/dev/ttyUSB0"/>
     <xacro:property name="use_sim" value="$(arg use_sim)"/>
-    <xacro:property name="canbus_base" value="$(arg canbus_base)"/>
-    <xacro:property name="canbus_arm" value="$(arg canbus_arm)"/>
-    <xacro:property name="serial_port" value="$(arg serial_port)"/>
+    <xacro:property name="canbus_base" default="can0"/>
+    <xacro:property name="canbus_arm" default="can1"/>
+    <xacro:property name="serial_port" default="/dev/ttyUSB0"/>
     <xacro:nxp_omniman />
     <!-- ============================================================

Commit message: Fixing can bus problem, can bus usb also has been fixed by changing can bus unique id.

File: omniman_ros2_control/description/nxp_omniman.urdf.xacro (robot description, xacro)
@@ -9,6 +9,6 @@
     <xacro:arg name="use_sim" default="false"/>
     <xacro:property name="use_sim" value="$(arg use_sim)"/>
-    <xacro:property name="canbus_base" default="can0"/>
-    <xacro:property name="canbus_arm" default="can1"/>
+    <xacro:property name="canbus_base" default="can_base"/>
+    <xacro:property name="canbus_arm" default="can_arm"/>
     <xacro:property name="serial_port" default="/dev/ttyUSB0"/>
     <xacro:nxp_omniman />

Commit message: Update udev rules for rplidar and dynamixel hardware

File: omniman_ros2_control/description/nxp_omniman.urdf.xacro (robot description, xacro)
@@ -11,5 +11,5 @@
     <xacro:property name="canbus_base" default="can_base"/>
     <xacro:property name="canbus_arm" default="can_arm"/>
-    <xacro:property name="serial_port" default="/dev/ttyUSB0"/>
+    <xacro:property name="serial_port" default="/dev/dynamixel"/>
     <xacro:nxp_omniman />
     <!-- ============================================================
