Commit message: Update Successfully Implemented SLAM toolbox for robot mapping and localization with occupancy grid mapping

File: omniman_description/urdf/omniman.urdf.xacro (robot description, xacro)
@@ -31,4 +31,30 @@
             </inertial>
         </link>
+        <!-- ==================== Lidar ==================== -->
+        <link name="lidar_link">
+            <visual>
+                <geometry>
+                    <mesh filename="package://omniman_description/meshes/visual/Lidar/Lidar_link.STL" />
+                </geometry>
+                <material name="grey" />
+            </visual>
+            <collision>
+                <geometry>
+                    <mesh filename="package://omniman_description/meshes/visual/Lidar/Lidar_link.STL" />
+                </geometry>
+            </collision>
+            <inertial>
+                <mass value="0.446536" />
+                <origin xyz="-0.000565 -0.000015 0.019299" rpy="0 0 0" />
+                <inertia ixx="0.000213" ixy="0.000000" ixz="-0.000006"
+                         iyy="0.000203" iyz="0.000000"
+                         izz="0.000297" />
+            </inertial>
+        </link>
+        <joint name="lidar_fixed_joint" type="fixed">
+            <parent link="base_link" />
+            <child link="lidar_link" />
+            <origin xyz="-0.042 0.000 0.075" rpy="0 0 0" />
+        </joint>
         <!-- ==================== Front_left Wheel ==================== -->
         <joint name="Front_left_couple_fixed_joint" type="fixed">

Commit message: Adding Documentation and Updating Configurations for simulation

File: omniman_description/urdf/omniman.urdf.xacro (robot description, xacro)
@@ -4,5 +4,5 @@
         <color rgba="0.5 0.5 0.5 1.0" />
     </material>
-    <xacro:macro name="nxp_omniman" >
+    <xacro:macro name="nxp_omniman" params="use_sim:=false">
         <link name="base_footprint" />
         <joint name="base_footprint_joint" type="fixed">
@@ -55,5 +55,10 @@
             <parent link="base_link" />
             <child link="lidar_link" />
-            <origin xyz="-0.042 0.000 0.078" rpy="0 0 3.14159" />
+            <xacro:if value="${use_sim}">
+                <origin xyz="-0.042 0.000 0.078" rpy="0 0 0" />
+            </xacro:if>
+            <xacro:unless value="${use_sim}">
+                <origin xyz="-0.042 0.000 0.078" rpy="0 0 3.14159" />
+            </xacro:unless>
         </joint>
         <!-- ==================== Front_left Wheel ==================== -->

File: omniman_ros2_control/description/nxp_omniman.urdf.xacro (robot description, xacro)
@@ -12,5 +12,5 @@
     <xacro:property name="canbus_arm" default="can_arm"/>
     <xacro:property name="serial_port" default="/dev/dynamixel"/>
-    <xacro:nxp_omniman />
+    <xacro:nxp_omniman use_sim="${use_sim}" />
     <!-- ============================================================
          Isaac Sim mock hardware (TopicBasedSystem)
