Commit message: Changing URDF direction doesn't correct

File: omniman_description/urdf/omniman.urdf (robot description, URDF)
Before this commit: robot nxp_omniman, 55 links, 54 joints
Joints:
- joint palm_yaw_joint: axis 0 0 -1 -> 0 0 1

File: omniman_description/urdf/omniman.urdf.xacro (robot description, xacro)
@@ -1315,5 +1315,5 @@
             <child link="palm_link" />
             <origin xyz="0.000 -0.019 0.064" rpy="0 0 0" />
-            <axis xyz="0 0 -1" />
+            <axis xyz="0 0 1" />
             <limit effort="10" velocity="1.0" lower="-3.14" upper="3.14" />
         </joint>

Commit message: Adding lidar to isaac sim simulation and ros2 control configuration

File: omniman_description/urdf/omniman.urdf (robot description, URDF)
Before this commit: robot nxp_omniman, 55 links, 54 joints
Links:
- added link lidar_link, mass 0.446536; collision mesh filename=package://omniman_description/meshes/visual/Lidar/Lidar_lin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; visual mesh filename=package://omniman_description/meshes/visual/Lidar/Lidar_lin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
Joints:
- added joint lidar_fixed_joint: type fixed, parent base_link, child lidar_link, origin xyz=-0.042 0.000 0.075 rpy=0 0 0

File: omniman_ros2_control/description/nxp_omniman.urdf.xacro (robot description, xacro)
@@ -18,11 +18,10 @@
          ============================================================ -->
     <xacro:if value="${use_sim}">
-        <ros2_control name="OmnimanSimSystem" type="system">
+        <ros2_control name="SimWheels" type="system">
             <hardware>
                 <plugin>topic_based_ros2_control/TopicBasedSystem</plugin>
-                <param name="joint_commands_topic">/isaac_joint_commands</param>
-                <param name="joint_states_topic">/isaac_joint_states</param>
+                <param name="joint_commands_topic">/isaac_wheel_commands</param>
+                <param name="joint_states_topic">/isaac_wheel_states</param>
             </hardware>
-            <!-- Mecanum wheels -->
             <joint name="Front_left_plate_continuous_joint">
                 <command_interface name="velocity"/>
@@ -45,5 +44,11 @@
                 <state_interface name="velocity"/>
             </joint>
-            <!-- Arm joints -->
+        </ros2_control>
+        <ros2_control name="SimArm" type="system">
+            <hardware>
+                <plugin>topic_based_ros2_control/TopicBasedSystem</plugin>
+                <param name="joint_commands_topic">/isaac_arm_commands</param>
+                <param name="joint_states_topic">/isaac_arm_states</param>
+            </hardware>
             <joint name="shoulder_yaw_joint">
                 <command_interface name="position"/>

Commit message: Update lidar link collide with base (under development)

File: omniman_description/urdf/omniman.urdf (robot description, URDF)
Before this commit: robot nxp_omniman, 56 links, 55 joints
Joints:
- joint lidar_fixed_joint: origin xyz=-0.042 0.000 0.075 rpy=0 0 0 -> xyz=-0.042 0.000 0.078 rpy=0 0 0

File: omniman_description/urdf/omniman.urdf.xacro (robot description, xacro)
@@ -55,5 +55,5 @@
             <parent link="base_link" />
             <child link="lidar_link" />
-            <origin xyz="-0.042 0.000 0.075" rpy="0 0 0" />
+            <origin xyz="-0.042 0.000 0.080" rpy="0 0 0" />
         </joint>
         <!-- ==================== Front_left Wheel ==================== -->

Commit message: Update lidar_link position in URDF, this still under development or testing

File: omniman_description/urdf/omniman.urdf (robot description, URDF)
Before this commit: robot nxp_omniman, 56 links, 55 joints
Joints:
- joint lidar_fixed_joint: origin xyz=-0.042 0.000 0.078 rpy=0 0 0 -> xyz=-0.042 0.000 0.080 rpy=0 0 0

File: omniman_description/urdf/omniman.urdf.xacro (robot description, xacro)
@@ -55,5 +55,5 @@
             <parent link="base_link" />
             <child link="lidar_link" />
-            <origin xyz="-0.042 0.000 0.080" rpy="0 0 0" />
+            <origin xyz="-0.042 0.000 0.078" rpy="0 0 0" />
         </joint>
         <!-- ==================== Front_left Wheel ==================== -->

Commit message: Update urdf lidar link that inverted 180degree

File: omniman_description/urdf/omniman.urdf (robot description, URDF)
Before this commit: robot nxp_omniman, 56 links, 55 joints
Joints:
- joint lidar_fixed_joint: origin xyz=-0.042 0.000 0.080 rpy=0 0 0 -> xyz=-0.042 0.000 0.080 rpy=0 0 3.14159

File: omniman_description/urdf/omniman.urdf.xacro (robot description, xacro)
@@ -55,5 +55,5 @@
             <parent link="base_link" />
             <child link="lidar_link" />
-            <origin xyz="-0.042 0.000 0.078" rpy="0 0 0" />
+            <origin xyz="-0.042 0.000 0.078" rpy="0 0 3.14159" />
         </joint>
         <!-- ==================== Front_left Wheel ==================== -->

Commit message: Update TCP at the inner surfaces of the two fingertips meet.

File: omniman_description/urdf/omniman.urdf (robot description, URDF)
Before this commit: robot nxp_omniman, 56 links, 55 joints
Joints:
- joint ee_joint: origin xyz=0.000 0.000 0.1 rpy=0 0 0 -> xyz=0.000 0.000 0.080 rpy=0 0 0

File: omniman_description/urdf/omniman.urdf.xacro (robot description, xacro)
@@ -1427,5 +1427,5 @@
             <parent link="palm_link" />
             <child link="ee_link" />
-            <origin xyz="0.000 0.000 0.1" rpy="0 0 0" />
+            <origin xyz="0.000 0.000 0.080" rpy="0 0 0" />
         </joint>
         <link name="ee_link" />

File: omniman_description/urdf/omniman_isaac.urdf (robot description, URDF)
Before this commit: robot nxp_omniman, 56 links, 55 joints
Joints:
- joint ee_joint: origin xyz=0.000 0.000 0.1 rpy=0 0 0 -> xyz=0.000 0.000 0.080 rpy=0 0 0

Commit message: Update lidar link position

File: omniman_description/urdf/omniman.urdf (robot description, URDF)
Before this commit: robot nxp_omniman, 56 links, 55 joints
Joints:
- joint lidar_fixed_joint: origin xyz=-0.042 0.000 0.080 rpy=0 0 3.14159 -> xyz=-0.070 0.000 0.077 rpy=0 0 0

File: omniman_description/urdf/omniman.urdf.xacro (robot description, xacro)
@@ -56,8 +56,8 @@
             <child link="lidar_link" />
             <xacro:if value="${use_sim}">
-                <origin xyz="-0.042 0.000 0.078" rpy="0 0 0" />
+                <origin xyz="-0.070 0.000 0.077" rpy="0 0 0" />
             </xacro:if>
             <xacro:unless value="${use_sim}">
-                <origin xyz="-0.042 0.000 0.078" rpy="0 0 3.14159" />
+                <origin xyz="-0.070 0.000 0.077" rpy="0 0 0" />
             </xacro:unless>
         </joint>

Commit message: Update Velocity Threshold

File: omniman_description/urdf/omniman.urdf (robot description, URDF)
Before this commit: robot nxp_omniman, 56 links, 55 joints
Joints:
- joint arm_yaw_joint: limit lower=-3.14 upper=3.14 effort=10 velocity=1.0 -> lower=-3.14 upper=3.14 effort=10 velocity=3.0
- joint forearm_pitch_joint: limit lower=-2.33 upper=2.4 effort=10 velocity=1.0 -> lower=-2.33 upper=2.4 effort=10 velocity=3.0
- joint palm_yaw_joint: limit lower=-3.14 upper=3.14 effort=10 velocity=1.0 -> lower=-3.14 upper=3.14 effort=10 velocity=3.0
- joint shoulder_yaw_joint: limit lower=-3.14 upper=3.14 effort=10 velocity=1.0 -> lower=-3.14 upper=3.14 effort=10 velocity=3.0
- joint upper_shoulder_pitch_joint: limit lower=-1.70 upper=1.70 effort=10 velocity=1.0 -> lower=-1.70 upper=1.70 effort=10 velocity=3.0
- joint wrist_pitch_joint: limit lower=-1.86 upper=1.69 effort=10 velocity=1.0 -> lower=-1.86 upper=1.69 effort=10 velocity=3.0

File: omniman_description/urdf/omniman.urdf.xacro (robot description, xacro)
@@ -1212,5 +1212,5 @@
             <origin xyz="0.082 0.000 0.129" rpy="0 0 0" />
             <axis xyz="0 0 -1" />
-            <limit effort="10" velocity="1.0" lower="-3.14" upper="3.14" />
+            <limit effort="10" velocity="3.0" lower="-3.14" upper="3.14" />
         </joint>
         <link name="shoulder_link">
@@ -1239,5 +1239,5 @@
             <origin xyz="0.0 0.034 0.045" rpy="0 0 0" />
             <axis xyz="0 -1 0" />
-            <limit effort="10" velocity="1.0" lower="-1.70" upper="1.70" />
+            <limit effort="10" velocity="3.0" lower="-1.70" upper="1.70" />
         </joint>
         <link name="upper_shoulder_link">
@@ -1266,5 +1266,5 @@
             <origin xyz="0.0 -0.036 0.103" rpy="0 0 0" />
             <axis xyz="0 0 -1" />
-            <limit effort="10" velocity="1.0" lower="-3.14" upper="3.14" />
+            <limit effort="10" velocity="3.0" lower="-3.14" upper="3.14" />
         </joint>
         <link name="arm_link">
@@ -1293,5 +1293,5 @@
             <origin xyz="0.0 0.034 0.045" rpy="0 0 0" />
             <axis xyz="0 -1 0" />
-            <limit effort="10" velocity="1.0" lower="-2.33" upper="2.4" />
+            <limit effort="10" velocity="3.0" lower="-2.33" upper="2.4" />
         </joint>
         <link name="forearm_link">
@@ -1320,5 +1320,5 @@
             <origin xyz="0.0 -0.017 0.100" rpy="0 0 0" />
             <axis xyz="0 1 0" />
-            <limit effort="10" velocity="1.0" lower="-1.86" upper="1.69" />
+            <limit effort="10" velocity="3.0" lower="-1.86" upper="1.69" />
         </joint>
         <link name="wrist_link">
@@ -1347,5 +1347,5 @@
             <origin xyz="0.000 -0.019 0.064" rpy="0 0 0" />
             <axis xyz="0 0 1" />
-            <limit effort="10" velocity="1.0" lower="-3.14" upper="3.14" />
+            <limit effort="10" velocity="3.0" lower="-3.14" upper="3.14" />
         </joint>
         <link name="palm_link">

Commit message: Add Camera link

File: omniman_description/urdf/omniman.urdf (robot description, URDF)
Before this commit: robot nxp_omniman, 56 links, 55 joints
Links:
- added link camera_link, mass 0.312030; collision mesh filename=package://omniman_description/meshes/visual/Camera/Camera_l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; visual mesh filename=package://omniman_description/meshes/visual/Camera/Camera_l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
Joints:
- added joint camera_fixed_joint: type fixed, parent palm_link, child camera_link, origin xyz=0.008 -0.021 0.006 rpy=0 0 0

File: omniman_description/urdf/omniman.urdf.xacro (robot description, xacro)
@@ -1369,4 +1369,30 @@
             </inertial>
         </link>
+        <!-- ==================== Camera =================== -->
+        <link name="camera_link">
+            <visual>
+                <geometry>
+                    <mesh filename="package://omniman_description/meshes/visual/Camera/Camera_link.STL" />
+                </geometry>
+                <material name="grey" />
+            </visual>
+            <collision>
+                <geometry>
+                    <mesh filename="package://omniman_description/meshes/visual/Camera/Camera_link.STL" />
+                </geometry>
+            </collision>
+            <inertial>
+                <mass value="0.312030" />
+                <origin xyz="-0.056976 0.020980 0.034842" rpy="0 0 0" />
+                <inertia ixx="0.000262" ixy="0.000000" ixz="-0.000079"
+                        iyy="0.000228" iyz="0.000000"
+                        izz="0.000228" />
+            </inertial>
+        </link>
+    <joint name="camera_fixed_joint" type="fixed">
+        <parent link="palm_link" />
+        <child link="camera_link" />
+        <origin xyz="0.008 -0.021 0.006" rpy="0 0 0" />
+    </joint>
         <joint name="left_finger_prismatic_joint" type="prismatic">
             <parent link="palm_link" />

File: omniman_description/urdf/omniman_isaac.urdf (robot description, URDF)
Before this commit: robot nxp_omniman, 56 links, 55 joints
Links:
- added link camera_link, mass 0.312030; collision mesh filename=package://omniman_description/meshes/visual/Camera/Camera_l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; visual mesh filename=package://omniman_description/meshes/visual/Camera/Camera_l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
Joints:
- added joint camera_fixed_joint: type fixed, parent palm_link, child camera_link, origin xyz=0.008 -0.021 0.006 rpy=0 0 0
- joint ee_joint: origin xyz=0.000 0.000 0.080 rpy=0 0 0 -> xyz=0 0 0.080 rpy=0 0 0; type continuous -> fixed

Commit message: Update new environment for testing new mediapipe feature

File: omniman_description/urdf/omniman.urdf (robot description, URDF)
Before this commit: robot nxp_omniman, 57 links, 56 joints
Links:
- added link camera_optical_frame
Joints:
- added joint camera_optical_fixed_joint: type fixed, parent camera_link, child camera_optical_frame, origin xyz=-0.071 0.021 0.059 rpy=0 0 -1.5707963

File: omniman_description/urdf/omniman.urdf.xacro (robot description, xacro)
@@ -1370,4 +1370,9 @@
         </link>
         <!-- ==================== Camera =================== -->
+        <joint name="camera_fixed_joint" type="fixed">
+            <parent link="palm_link" />
+            <child link="camera_link" />
+            <origin xyz="0.008 -0.021 0.006" rpy="0 0 0" />
+        </joint>
         <link name="camera_link">
             <visual>
@@ -1390,9 +1395,10 @@
             </inertial>
         </link>
-    <joint name="camera_fixed_joint" type="fixed">
-        <parent link="palm_link" />
-        <child link="camera_link" />
-        <origin xyz="0.008 -0.021 0.006" rpy="0 0 0" />
-    </joint>
+        <joint name="camera_optical_fixed_joint" type="fixed">
+            <parent link="camera_link" />
+            <child link="camera_optical_frame" />
+            <origin xyz="-0.071 0.021 0.059" rpy="0 0 -1.5707963" />
+        </joint>
+        <link name="camera_optical_frame" />
         <joint name="left_finger_prismatic_joint" type="prismatic">
             <parent link="palm_link" />
