Commit message: Update readme vla-training.md.
Update URDF base_footprint computed from wheel radius (0.05m) + where the wheel axle sits (0.043) = 0.093m.

Update launch file to launch teleop for inference and add stop order between nav2 and inference

Update introduce laser filters mechanism,
LaserScanPolygonFilter (your real footprint, geometrically correct) plus LaserScanSpeckleFilter
for single-beam noise.

File: omniman_description/urdf/omniman.urdf (robot description, URDF)
Before this commit: robot nxp_omniman, 58 links, 57 joints
Joints:
- joint base_footprint_joint: origin xyz=0 0 0.09 rpy=0 0 0 -> xyz=0 0 0.093 rpy=0 0 0

File: omniman_description/urdf/omniman.urdf.xacro (robot description, xacro)
@@ -9,5 +9,5 @@
             <parent link="base_footprint" />
             <child link="base_link" />
-            <origin xyz="0 0 0.09" rpy="0 0 0" />
+            <origin xyz="0 0 0.093" rpy="0 0 0" />
         </joint>
         <link name="base_link">
