Commit message: Update ros2 hardware integration: current limit for tuning moveit teleoperation

File: dynamixel_hardware/dynamixel_hardware_interface/ros2_control/dynamixel_motor.ros2_control.xacro (robot description, xacro)
@@ -1,5 +1,5 @@
 <?xml version="1.0"?>
 <robot xmlns:xacro="http://www.ros.org/wiki/xacro">
-    <xacro:macro name="dynamixel_ros2_control" params="name serial_device device_id joint_name use_prismatic:=0 revolute_max:=0.0 revolute_min:=0.0 prismatic_max:=0.0 prismatic_min:=0.0 driver_mode:=0">
+    <xacro:macro name="dynamixel_ros2_control" params="name serial_device device_id joint_name use_prismatic:=0 revolute_max:=0.0 revolute_min:=0.0 prismatic_max:=0.0 prismatic_min:=0.0 driver_mode:=0 current_limit:=300 profile_velocity:=0 profile_acceleration:=0">
         <ros2_control name="${name}" type="system">
             <hardware>
@@ -46,9 +46,9 @@
                 <param name="Position I Gain">100</param>
                 <param name="Position D Gain">100</param>
-                <param name="Profile Velocity">0</param>
-                <param name="Profile Acceleration">0</param>
+                <param name="Profile Velocity">${profile_velocity}</param>
+                <param name="Profile Acceleration">${profile_acceleration}</param>
                 <param name="Drive Mode">${driver_mode}</param>
                 <param name="Return Delay Time">2</param>
-                <param name="Current Limit">300</param>
+                <param name="Current Limit">${current_limit}</param>
             </gpio>
             <transmission name="${joint_name}_transmission">

File: omniman_ros2_control/description/nxp_omniman.urdf.xacro (robot description, xacro)
@@ -134,11 +134,14 @@
         <xacro:robstride_ros2_control name="ForearmPitch" canbus="${canbus_arm}" device_id="8" joint_name="forearm_pitch_joint" axis_direction="1"/>
         <!-- ========== Wrist + Gripper (Dynamixel on serial_port) ========== -->
-        <xacro:dynamixel_ros2_control name="WristPitch" serial_device="${serial_port}" device_id="9" joint_name="wrist_pitch_joint"/>
-        <xacro:dynamixel_ros2_control name="PalmYaw" serial_device="${serial_port}" device_id="10" joint_name="palm_yaw_joint"/>
+        <xacro:dynamixel_ros2_control name="WristPitch" serial_device="${serial_port}" device_id="9" joint_name="wrist_pitch_joint"
+                                      current_limit="450"/>
+        <xacro:dynamixel_ros2_control name="PalmYaw" serial_device="${serial_port}" device_id="10" joint_name="palm_yaw_joint"
+                                      current_limit="300"/>
         <xacro:dynamixel_ros2_control name="LeftFingerPrismatic" serial_device="${serial_port}" device_id="11"
                                       joint_name="left_finger_prismatic_joint"
                                       use_prismatic="1"
                                       revolute_max="0.0" revolute_min="-2.5"
-                                      prismatic_max="0.019" prismatic_min="-0.013"/>
+                                      prismatic_max="0.019" prismatic_min="-0.013"
+                                      current_limit="100"/>
     </xacro:unless>
 </robot>

Commit message: Update ros2 hardware integration: PID parameter for teleoperation

File: dynamixel_hardware/dynamixel_hardware_interface/ros2_control/dynamixel_motor.ros2_control.xacro (robot description, xacro)
@@ -1,5 +1,5 @@
 <?xml version="1.0"?>
 <robot xmlns:xacro="http://www.ros.org/wiki/xacro">
-    <xacro:macro name="dynamixel_ros2_control" params="name serial_device device_id joint_name use_prismatic:=0 revolute_max:=0.0 revolute_min:=0.0 prismatic_max:=0.0 prismatic_min:=0.0 driver_mode:=0 current_limit:=300 profile_velocity:=0 profile_acceleration:=0">
+    <xacro:macro name="dynamixel_ros2_control" params="name serial_device device_id joint_name use_prismatic:=0 revolute_max:=0.0 revolute_min:=0.0 prismatic_max:=0.0 prismatic_min:=0.0 driver_mode:=0 current_limit:=300 profile_velocity:=0 profile_acceleration:=0 position_p_gain:=800 position_i_gain:=0 position_d_gain:=100">
         <ros2_control name="${name}" type="system">
             <hardware>
@@ -43,7 +43,7 @@
                 <state_interface name="Torque Enable"/>
                 <state_interface name="Present Input Voltage"/>
-                <param name="Position P Gain">800</param>
-                <param name="Position I Gain">100</param>
-                <param name="Position D Gain">100</param>
+                <param name="Position P Gain">${position_p_gain}</param>
+                <param name="Position I Gain">${position_i_gain}</param>
+                <param name="Position D Gain">${position_d_gain}</param>
                 <param name="Profile Velocity">${profile_velocity}</param>
                 <param name="Profile Acceleration">${profile_acceleration}</param>

File: omniman_ros2_control/description/nxp_omniman.urdf.xacro (robot description, xacro)
@@ -143,5 +143,6 @@
                                       revolute_max="0.0" revolute_min="-2.5"
                                       prismatic_max="0.019" prismatic_min="-0.013"
-                                      current_limit="100"/>
+                                      current_limit="100"
+                                      position_i_gain="100"/>
     </xacro:unless>
 </robot>

Commit message: Update ros2 dynamiel hardware interation parameters for wrist and palm to tune pid moveit servo teleoperation

File: dynamixel_hardware/dynamixel_hardware_interface/ros2_control/dynamixel_motor.ros2_control.xacro (robot description, xacro)
@@ -1,5 +1,5 @@
 <?xml version="1.0"?>
 <robot xmlns:xacro="http://www.ros.org/wiki/xacro">
-    <xacro:macro name="dynamixel_ros2_control" params="name serial_device device_id joint_name use_prismatic:=0 revolute_max:=0.0 revolute_min:=0.0 prismatic_max:=0.0 prismatic_min:=0.0 driver_mode:=0 current_limit:=300 profile_velocity:=0 profile_acceleration:=0 position_p_gain:=800 position_i_gain:=0 position_d_gain:=100">
+    <xacro:macro name="dynamixel_ros2_control" params="name serial_device device_id joint_name use_prismatic:=0 revolute_max:=0.0 revolute_min:=0.0 prismatic_max:=0.0 prismatic_min:=0.0 driver_mode:=0 current_limit:=300 profile_velocity:=200 profile_acceleration:=50 position_p_gain:=800 position_i_gain:=100 position_d_gain:=100">
         <ros2_control name="${name}" type="system">
             <hardware>

File: omniman_ros2_control/description/nxp_omniman.urdf.xacro (robot description, xacro)
@@ -136,9 +136,11 @@
         <xacro:dynamixel_ros2_control name="WristPitch" serial_device="${serial_port}" device_id="9" joint_name="wrist_pitch_joint"
                                       current_limit="800"
-                                      position_i_gain="500"
-                                      profile_velocity="500"
-                                      profile_acceleration="0"/>
+                                      position_p_gain="2300"
+                                      profile_velocity="0"
+                                      />
         <xacro:dynamixel_ros2_control name="PalmYaw" serial_device="${serial_port}" device_id="10" joint_name="palm_yaw_joint"
-                                      current_limit="800"/>
+                                      current_limit="800"
+                                      profile_velocity="0"
+                                      />
         <xacro:dynamixel_ros2_control name="LeftFingerPrismatic" serial_device="${serial_port}" device_id="11"
                                       joint_name="left_finger_prismatic_joint"

Commit message: Update Dynamixel Hardware Integration parameters

File: dynamixel_hardware/dynamixel_hardware_interface/ros2_control/dynamixel_motor.ros2_control.xacro (robot description, xacro)
@@ -1,5 +1,5 @@
 <?xml version="1.0"?>
 <robot xmlns:xacro="http://www.ros.org/wiki/xacro">
-    <xacro:macro name="dynamixel_ros2_control" params="name serial_device device_id joint_name use_prismatic:=0 revolute_max:=0.0 revolute_min:=0.0 prismatic_max:=0.0 prismatic_min:=0.0 driver_mode:=0 current_limit:=300 profile_velocity:=200 profile_acceleration:=50 position_p_gain:=800 position_i_gain:=100 position_d_gain:=100">
+    <xacro:macro name="dynamixel_ros2_control" params="name serial_device device_id joint_name use_prismatic:=0 revolute_max:=0.0 revolute_min:=0.0 prismatic_max:=0.0 prismatic_min:=0.0 driver_mode:=0">
         <ros2_control name="${name}" type="system">
             <hardware>
@@ -43,12 +43,6 @@
                 <state_interface name="Torque Enable"/>
                 <state_interface name="Present Input Voltage"/>
-                <param name="Position P Gain">${position_p_gain}</param>
-                <param name="Position I Gain">${position_i_gain}</param>
-                <param name="Position D Gain">${position_d_gain}</param>
-                <param name="Profile Velocity">${profile_velocity}</param>
-                <param name="Profile Acceleration">${profile_acceleration}</param>
                 <param name="Drive Mode">${driver_mode}</param>
                 <param name="Return Delay Time">2</param>
-                <param name="Current Limit">${current_limit}</param>
             </gpio>
             <transmission name="${joint_name}_transmission">

Commit message: Update dynamixel motor p gain parameter

File: dynamixel_hardware/dynamixel_hardware_interface/ros2_control/dynamixel_motor.ros2_control.xacro (robot description, xacro)
@@ -1,5 +1,5 @@
 <?xml version="1.0"?>
 <robot xmlns:xacro="http://www.ros.org/wiki/xacro">
-    <xacro:macro name="dynamixel_ros2_control" params="name serial_device device_id joint_name use_prismatic:=0 revolute_max:=0.0 revolute_min:=0.0 prismatic_max:=0.0 prismatic_min:=0.0 driver_mode:=0">
+    <xacro:macro name="dynamixel_ros2_control" params="name serial_device device_id joint_name use_prismatic:=0 revolute_max:=0.0 revolute_min:=0.0 prismatic_max:=0.0 prismatic_min:=0.0 driver_mode:=0 position_p_gain:=800">
         <ros2_control name="${name}" type="system">
             <hardware>
@@ -43,4 +43,5 @@
                 <state_interface name="Torque Enable"/>
                 <state_interface name="Present Input Voltage"/>
+                <param name="Position P Gain">${position_p_gain}</param>
                 <param name="Drive Mode">${driver_mode}</param>
                 <param name="Return Delay Time">2</param>

File: omniman_ros2_control/description/nxp_omniman.urdf.xacro (robot description, xacro)
@@ -135,4 +135,5 @@
         <!-- ========== Wrist + Gripper (Dynamixel on serial_port) ========== -->
         <xacro:dynamixel_ros2_control name="WristPitch" serial_device="${serial_port}" device_id="9" joint_name="wrist_pitch_joint"
+                                      position_p_gain="2500"
                                       />
         <xacro:dynamixel_ros2_control name="PalmYaw" serial_device="${serial_port}" device_id="10" joint_name="palm_yaw_joint"
