Commit message: update the leader robot also should be have the original default values from robotis to prevent jitter, i think the pid that was there before, was the correct values but now the leader and follower has slightly delayed when we teleoperate.

File: dynamixel_hardware/dynamixel_hardware_interface/ros2_control/dynamixel_motor.ros2_control.xacro (robot description, xacro)
@@ -1,5 +1,5 @@
 <?xml version="1.0"?>
 <robot xmlns:xacro="http://www.ros.org/wiki/xacro">
-    <xacro:macro name="dynamixel_ros2_control" params="name serial_device device_id joint_name use_prismatic:=0 revolute_max:=0.0 revolute_min:=0.0 prismatic_max:=0.0 prismatic_min:=0.0 driver_mode:=0 position_p_gain:=800">
+    <xacro:macro name="dynamixel_ros2_control" params="name serial_device device_id joint_name use_prismatic:=0 revolute_max:=0.0 revolute_min:=0.0 prismatic_max:=0.0 prismatic_min:=0.0 driver_mode:=0">
         <ros2_control name="${name}" type="system">
             <hardware>

File: leader_ros2_control/description/leader_ros2_control.urdf.xacro (robot description, xacro)
@@ -13,5 +13,5 @@
          Drive Modes match leader.gravity.xacro: 1,0,1,1,1,0,0
          ============================================================ -->
-    <xacro:macro name="leader_dynamixel_ros2_control" params="name device_id joint_name driver_mode:=0 position_p_gain:=800">
+    <xacro:macro name="leader_dynamixel_ros2_control" params="name device_id joint_name driver_mode:=0">
         <ros2_control name="${name}" type="system">
             <hardware>
@@ -19,9 +19,10 @@
                 <param name="port_name">${serial_port}</param>
                 <param name="baud_rate">1000000</param>
-                <param name="error_timeout_ms">500</param>
+                <param name="error_timeout_ms">0.2</param>
                 <param name="disable_torque_at_init">true</param>
                 <param name="dynamixel_model_folder">/param/dxl_model</param>
                 <param name="number_of_joints">1</param>
                 <param name="number_of_transmissions">1</param>
+                <param name="ros_update_freq">200</param>
                 <param name="dynamixel_state_pub_msg_name">dynamixel_hardware_interface/dxl_state</param>
                 <param name="get_dynamixel_data_srv_name">dynamixel_hardware_interface/get_dxl_data</param>
@@ -45,8 +46,11 @@
                 <state_interface name="Torque Enable"/>
                 <state_interface name="Present Input Voltage"/>
-                <param name="Position P Gain">${position_p_gain}</param>
+                <param name="Position P Gain">800</param>
+                <param name="Position I Gain">100</param>
+                <param name="Position D Gain">100</param>
+                <param name="Profile Velocity">200</param>
+                <param name="Profile Acceleration">50</param>
                 <param name="Drive Mode">${driver_mode}</param>
-                <param name="Operating Mode">3</param>
-                <param name="Return Delay Time">2</param>
+                <param name="Return Delay Time">0</param>
             </gpio>
             <transmission name="${joint_name}_transmission">

Commit message: Update new configuration for dynamixel hardware integration, the gripper often overload, this happened when the gripper trying to close when there are object it grabs, so the position when it close doesn't match with the command, it sends so much current tying to reach that position, and it shutdown automatically when the current is exceed the limit that we define. so the solution is to add number 5 operating mode where it will adjust the current.
Update omniman_vla mission, we implemented check the home position of arm robot to switch between nav2 and policy inference

File: dynamixel_hardware/dynamixel_hardware_interface/ros2_control/dynamixel_motor.ros2_control.xacro (robot description, xacro)
@@ -1,5 +1,5 @@
 <?xml version="1.0"?>
 <robot xmlns:xacro="http://www.ros.org/wiki/xacro">
-    <xacro:macro name="dynamixel_ros2_control" params="name serial_device device_id joint_name use_prismatic:=0 revolute_max:=0.0 revolute_min:=0.0 prismatic_max:=0.0 prismatic_min:=0.0 driver_mode:=0">
+    <xacro:macro name="dynamixel_ros2_control" params="name serial_device device_id joint_name use_prismatic:=0 revolute_max:=0.0 revolute_min:=0.0 prismatic_max:=0.0 prismatic_min:=0.0 driver_mode:=0 operating_mode:='' goal_current:=''">
         <ros2_control name="${name}" type="system">
             <hardware>
@@ -50,4 +50,11 @@
                 <param name="Drive Mode">${driver_mode}</param>
                 <param name="Return Delay Time">0</param>
+                <!-- Optional, only emitted when set. Mode 5 is current based position, Goal Current caps grip force -->
+                <xacro:if value="${operating_mode != ''}">
+                    <param name="Operating Mode">${operating_mode}</param>
+                </xacro:if>
+                <xacro:if value="${goal_current != ''}">
+                    <param name="Goal Current">${goal_current}</param>
+                </xacro:if>
             </gpio>
             <transmission name="${joint_name}_transmission">

File: omniman_ros2_control/description/nxp_omniman.urdf.xacro (robot description, xacro)
@@ -143,4 +143,5 @@
                                       revolute_max="0.0" revolute_min="-2.5"
                                       prismatic_max="0.019" prismatic_min="-0.013"
+                                      operating_mode="5" goal_current="200"
                                       />
     </xacro:unless>

File: omniman_vla/description/nxp_omniman.urdf.xacro (robot description, xacro)
@@ -62,4 +62,5 @@
                                   revolute_max="0.0" revolute_min="-2.5"
                                   prismatic_max="0.019" prismatic_min="-0.013"
+                                  operating_mode="5" goal_current="200"
                                   />
 </robot>

Commit message: Update trying to lower the p gain, because after apply the previous commit change, now the gripper jitter back forth, It overshoots, reverses at full current, overshoots again. Before, in mode 3 with no current cap, it pushed through the friction and hid this.

File: dynamixel_hardware/dynamixel_hardware_interface/ros2_control/dynamixel_motor.ros2_control.xacro (robot description, xacro)
@@ -1,5 +1,5 @@
 <?xml version="1.0"?>
 <robot xmlns:xacro="http://www.ros.org/wiki/xacro">
-    <xacro:macro name="dynamixel_ros2_control" params="name serial_device device_id joint_name use_prismatic:=0 revolute_max:=0.0 revolute_min:=0.0 prismatic_max:=0.0 prismatic_min:=0.0 driver_mode:=0 operating_mode:='' goal_current:=''">
+    <xacro:macro name="dynamixel_ros2_control" params="name serial_device device_id joint_name use_prismatic:=0 revolute_max:=0.0 revolute_min:=0.0 prismatic_max:=0.0 prismatic_min:=0.0 driver_mode:=0 operating_mode:='' goal_current:='' position_p_gain:=800 profile_velocity:=0 profile_acceleration:=0">
         <ros2_control name="${name}" type="system">
             <hardware>
@@ -43,9 +43,9 @@
                 <state_interface name="Torque Enable"/>
                 <state_interface name="Present Input Voltage"/>
-                <param name="Position P Gain">800</param>
+                <param name="Position P Gain">${position_p_gain}</param>
                 <param name="Position I Gain">0</param>
                 <param name="Position D Gain">0</param>
-                <param name="Profile Velocity">0</param>
-                <param name="Profile Acceleration">0</param>
+                <param name="Profile Velocity">${profile_velocity}</param>
+                <param name="Profile Acceleration">${profile_acceleration}</param>
                 <param name="Drive Mode">${driver_mode}</param>
                 <param name="Return Delay Time">0</param>

File: omniman_ros2_control/description/nxp_omniman.urdf.xacro (robot description, xacro)
@@ -144,4 +144,5 @@
                                       prismatic_max="0.019" prismatic_min="-0.013"
                                       operating_mode="5" goal_current="200"
+                                      position_p_gain="400"
                                       />
     </xacro:unless>

File: omniman_vla/description/nxp_omniman.urdf.xacro (robot description, xacro)
@@ -63,4 +63,5 @@
                                   prismatic_max="0.019" prismatic_min="-0.013"
                                   operating_mode="5" goal_current="200"
+                                  position_p_gain="400"
                                   />
 </robot>
