Commit message: Adding Ros2_control hardware bringup for leader robot. need to be aware with Operating Mode at hardware interface system because mode 0 did not disable torque, while leader.gravity.xacro uses operating mode 0 which is Goal Current instead of Position

File: leader_ros2_control/description/leader.gravity.xacro (robot description, xacro)
@@ -1,4 +1,9 @@
 <?xml version="1.0"?>
-<robot xmlns:xacro="http://www.ros.org/wiki/xacro">
+<robot name="leader" xmlns:xacro="http://www.ros.org/wiki/xacro">
+  <!-- Include the leader arm URDF -->
+  <xacro:include filename="$(find leader_description)/urdf/leader.urdf.xacro"/>
+  <!-- Launch arguments -->
+  <xacro:arg name="port_name" default="/dev/dynamixel_leader"/>
+  <xacro:leader />
   <!--
     Leader arm hardware in CURRENT (torque) control mode for gravity compensation.
@@ -10,5 +15,5 @@
     - Current Limit caps motor torque during tuning (raw units; 400 ~= 1.08 A ~= 1.9 Nm)
   -->
-  <xacro:macro name="leader_system" params="name port_name:=/dev/ttyUSB1">
+  <xacro:macro name="leader_system" params="name port_name:=/dev/dynamixel_leader">
     <ros2_control name="${name}" type="system">
       <hardware>
@@ -98,4 +103,5 @@
         <param name="Return Delay Time">0</param>
         <param name="Current Limit">400</param>
+        <param name="Goal Current">0</param>
       </gpio>
       <gpio name="dxl2">
@@ -110,4 +116,5 @@
         <param name="Return Delay Time">0</param>
         <param name="Current Limit">400</param>
+        <param name="Goal Current">0</param>
       </gpio>
       <gpio name="dxl3">
@@ -122,4 +129,5 @@
         <param name="Return Delay Time">0</param>
         <param name="Current Limit">400</param>
+        <param name="Goal Current">0</param>
       </gpio>
       <gpio name="dxl4">
@@ -134,4 +142,5 @@
         <param name="Return Delay Time">0</param>
         <param name="Current Limit">400</param>
+        <param name="Goal Current">0</param>
       </gpio>
       <gpio name="dxl5">
@@ -146,4 +155,5 @@
         <param name="Return Delay Time">0</param>
         <param name="Current Limit">400</param>
+        <param name="Goal Current">0</param>
       </gpio>
       <gpio name="dxl6">
@@ -158,4 +168,5 @@
         <param name="Return Delay Time">0</param>
         <param name="Current Limit">400</param>
+        <param name="Goal Current">0</param>
       </gpio>
       <gpio name="dxl7">
@@ -170,6 +181,9 @@
         <param name="Return Delay Time">0</param>
         <param name="Current Limit">200</param>
+        <param name="Goal Current">0</param>
       </gpio>
     </ros2_control>
   </xacro:macro>
+  <!-- single dynamixel system: all 7 motors, effort command (Goal Current) -->
+  <xacro:leader_system name="leader_system" port_name="$(arg port_name)"/>
 </robot>
