Commit message: Update URDF, I have measured each part per part of the robot and calculate it in solidwork the center of mass, inertia dan mass.
Update gravity Compensation Controller parameters,
i have tune each joint parameter and observe the best behaviour that i can achieve

Update to show rviz robot visual
in order to avoid fight with omniman robot, we prepends '/leader' at every TF with using frame_prefix in launch.

File: leader_description/urdf/leader.urdf (robot description, URDF)
Before this commit: robot leader, 9 links, 8 joints
Links:
- link arm_link: mass 0.161017 -> 0.198517
- link forearm_link: mass 0.126166 -> 0.120758
- link palm_link: mass 0.141693 -> 0.167758
- link shoulder_link: mass 0.067330 -> 0.104932
- link upper_shoulder_link: mass 0.060696 -> 0.098298
- link wrist_link: mass 0.047237 -> 0.091000
Joints:
- joint forearm_pitch_joint: origin xyz=0.254 0.019 0.019 rpy=0 0 0 -> xyz=0.000 0.019 0.159 rpy=0 0 0
- joint wrist_pitch_joint: origin xyz=0.225 -0.002 0.000 rpy=0 0 0 -> xyz=0.000 -0.002 0.135 rpy=0 0 0

File: leader_description/urdf/leader.urdf.xacro (robot description, xacro)
@@ -45,9 +45,9 @@
             </collision>
             <inertial>
-                <mass value="0.067330" />
-                <origin xyz="-0.011831 -0.004951 0.018905" rpy="0 0 0" />
-                <inertia ixx="0.000015" ixy="0.000000" ixz="0.0000000"
-                        iyy="0.000026" iyz="0.000000"
-                        izz="0.000024" />
+                <mass value="0.104932" />
+                <origin xyz="-0.011744 -0.003190 0.018889" rpy="0 0 0" />
+                <inertia ixx="0.000022" ixy="0.000000" ixz="0.0000000"
+                        iyy="0.000036" iyz="0.000000"
+                        izz="0.000034" />
             </inertial>
         </link>
@@ -72,9 +72,9 @@
             </collision>
             <inertial>
-                <mass value="0.060696" />
-                <origin xyz="0.000023 -0.018562 0.018781" rpy="0 0 0" />
-                <inertia ixx="0.000025" ixy="0.000000" ixz="0.000000"
-                        iyy="0.000021" iyz="0.000000"
-                        izz="0.000012" />
+                <mass value="0.098298" />
+                <origin xyz="0.000000 -0.018677 0.016030" rpy="0 0 0" />
+                <inertia ixx="0.000037" ixy="0.000000" ixz="0.000000"
+                        iyy="0.000032" iyz="0.000000"
+                        izz="0.000018" />
             </inertial>
         </link>
@@ -99,9 +99,9 @@
             </collision>
             <inertial>
-                <mass value="0.161017" />
-                <origin xyz="0.127050 0.000149 0.018851" rpy="0 0 0" />
-                <inertia ixx="0.000024" ixy="0.000003" ixz="0.000003"
-                        iyy="0.001502" iyz="0.000000"
-                        izz="0.001502" />
+                <mass value="0.198517" />
+                <origin xyz="0.004663 0.000160 0.082369" rpy="0 0 0" />
+                <inertia ixx="0.000775" ixy="0.000000" ixz="-0.000059"
+                        iyy="0.000786" iyz="0.000002"
+                        izz="0.000047" />
             </inertial>
         </link>
@@ -109,5 +109,5 @@
             <parent link="arm_link" />
             <child link="forearm_link" />
-            <origin xyz="0.254 0.019 0.019" rpy="0 0 0" />
+            <origin xyz="0.000 0.019 0.159" rpy="0 0 0" />
             <axis xyz="0 -1 0" />
             <limit effort="10" velocity="3.0" lower="-2.33" upper="2.4" />
@@ -126,9 +126,9 @@
             </collision>
             <inertial>
-                <mass value="0.126166" />
-                <origin xyz="0.137015 0.016972 -0.000011" rpy="0 0 0" />
-                <inertia ixx="0.000018" ixy="0.000004" ixz="0.000000"
-                        iyy="0.000810" iyz="0.000000"
-                        izz="0.000814" />
+                <mass value="0.120758" />
+                <origin xyz="0.000000 0.016998 0.099892" rpy="0 0 0" />
+                <inertia ixx="0.000231" ixy="0.000000" ixz="0.000000"
+                        iyy="0.000226" iyz="0.000002"
+                        izz="0.000021" />
             </inertial>
         </link>
@@ -136,5 +136,5 @@
             <parent link="forearm_link" />
             <child link="wrist_link" />
-            <origin xyz="0.225 -0.002 0.000" rpy="0 0 0" />
+            <origin xyz="0.000 -0.002 0.135" rpy="0 0 0" />
             <axis xyz="0 1 0" />
             <limit effort="10" velocity="3.0" lower="-1.86" upper="1.69" />
@@ -153,9 +153,9 @@
             </collision>
             <inertial>
-                <mass value="0.047237" />
-                <origin xyz="-0.000029 -0.027699 0.000563" rpy="0 0 0" />
-                <inertia ixx="0.000015" ixy="0.000000" ixz="0.000000"
-                        iyy="0.000008" iyz="0.000000"
-                        izz="0.000013" />
+                <mass value="0.091000" />
+                <origin xyz="0.000000 -0.027250 0.000360" rpy="0 0 0" />
+                <inertia ixx="0.000028" ixy="0.000000" ixz="0.000000"
+                        iyy="0.000015" iyz="0.000000"
+                        izz="0.000024" />
             </inertial>
         </link>
@@ -180,9 +180,9 @@
             </collision>
             <inertial>
-                <mass value="0.141693" />
-                <origin xyz="0.028024 0.008156 0.079739" rpy="0 0 0" />
-                <inertia ixx="0.000288" ixy="-0.000010" ixz="0.000010"
-                        iyy="0.000385" iyz="0.000054"
-                        izz="0.000158" />
+                <mass value="0.167758" />
+                <origin xyz="0.025752 0.013110 0.095377" rpy="0 0 0" />
+                <inertia ixx="0.000295" ixy="-0.000011" ixz="-0.000004"
+                        iyy="0.000363" iyz="0.000062"
+                        izz="0.000136" />
             </inertial>
         </link>

Commit message: Update Leader Follower Teleoperation has been implemented successfully. Added new launch file teleop_bridges_launch.py to launch the teleoperation system (both robot should bring up first and make sure it is in safe position) Added new script gripper teleop_bridge.py to control the gripper, because gripper has different controller, unit and name joint, so we should map this with independent node

File: leader_description/urdf/leader.urdf (robot description, URDF)
Before this commit: robot leader, 9 links, 8 joints
Joints:
- joint gripper_prismatic_joint: limit lower=-0.4 upper=1 effort=1 velocity=4.8 -> lower=-0.4 upper=0.0 effort=1 velocity=4.8

File: leader_description/urdf/leader.urdf.xacro (robot description, xacro)
@@ -192,5 +192,5 @@
             <origin xyz="0.033 0.004 0.127" rpy="0 0 0" />
             <axis xyz="0 -1 0" />
-            <limit effort="1" velocity="4.8" lower="-0.4" upper="1" />
+            <limit effort="1" velocity="4.8" lower="-0.4" upper="0.0" />
         </joint>
         <link name="gripper_link">
