Commit message: Added new package dedicated omniman_vla for VLA training with Physical AI Tools: - this package load everything that needed by physical ai tools, and leave the base wheels off. - i removed every simulation related code
Removed gripper_teleop_bridge.py:
- since now omniman_vla has mirrored gripper like leader, which what the physical ai tools need.
- we directly set the parameters for gripper in config yaml file

File: omniman_vla/urdf/omniman_vla.urdf.xacro (robot description, xacro)
@@ -24,5 +24,5 @@
             </collision>
             <inertial>
-                <mass value="11.60351" />
+                <mass value="11.503663" />
                 <origin xyz="0.007471 -0.002650 0.013517" rpy="0 0 0" />
                 <inertia ixx="0.130641" ixy="-0.005256" ixz="0.002401"
@@ -1401,5 +1401,5 @@
         </joint>
         <link name="camera_optical_frame" />
-        <joint name="left_finger_prismatic_joint" type="prismatic">
+        <joint name="gripper_prismatic_joint" type="prismatic">
             <parent link="palm_link" />
             <child link="left_finger_link" />
@@ -1409,5 +1409,5 @@
         </joint>
         <joint name="right_finger_prismatic_joint" type="prismatic">
-            <mimic joint="left_finger_prismatic_joint" multiplier="-1.0" offset="0.0" />
+            <mimic joint="gripper_prismatic_joint" multiplier="-1.0" offset="0.0" />
             <parent link="palm_link" />
             <child link="right_finger_link" />
