Commit message: Update the urdf xacro file to include all the wheels link

File: omniman_vla/urdf/omniman.urdf.xacro (robot description, xacro)
@@ -83,4 +83,264 @@
             </inertial>
         </link>
+        <link name="Front_left_plate_link">
+            <visual>
+                <geometry>
+                    <mesh filename="package://omniman_description/meshes/visual/Front_left_wheel/Front_left_plate_link.STL" />
+                </geometry>
+                <material name="grey" />
+            </visual>
+            <collision>
+                <geometry>
+                    <mesh filename="package://omniman_description/meshes/visual/Front_left_wheel/Front_left_plate_link.STL" />
+                </geometry>
+            </collision>
+            <inertial>
+                <mass value="0.330894" />
+                <origin xyz="0.000000 0.025959 0.000000" rpy="0 0 0" />
+                <inertia ixx="0.000188" ixy="0.000000" ixz="0.000000"
+                        iyy="0.000187" iyz="0.000000"
+                        izz="0.000188" />
+            </inertial>
+        </link>
+        <joint name="Front_left_plate_continuous_joint" type="continuous">
+            <parent link="Front_left_couple_link" />
+            <child link="Front_left_plate_link" />
+            <origin xyz="0 0.01729 0" rpy="0 0 0" />
+            <axis xyz="0 1 0" />
+        </joint>
+        <link name="Front_left_roller_link1">
+            <visual>
+                <geometry>
+                    <mesh filename="package://omniman_description/meshes/visual/Front_left_wheel/Front_left_roller_link1.STL" />
+                </geometry>
+                <material name="grey" />
+            </visual>
+            <collision>
+                <geometry>
+                    <mesh filename="package://omniman_description/meshes/visual/Front_left_wheel/Front_left_roller_link1.STL" />
+                </geometry>
+            </collision>
+            <inertial>
+                <mass value="0.009948" />
+                <origin xyz="0.000000 0.000000 0.000000" rpy="0 0 0" />
+                <inertia ixx="0.000001" ixy="0.000000" ixz="0.000000"
+                        iyy="0.000002" iyz="0.000000"
+                        izz="0.000002" />
+            </inertial>
+        </link>
+        <joint name="Front_left_roller_continuous_joint1" type="fixed">
+            <parent link="Front_left_plate_link" />
+            <child link="Front_left_roller_link1" />
+            <origin xyz="-0.0077812 0.025962 0.037903" rpy="-2.68 -0.14308 0.79578" />
+            <axis xyz="1 0 0" />
+        </joint>
+        <link name="Front_left_roller_link2">
+            <visual>
+                <geometry>
+                    <mesh filename="package://omniman_description/meshes/visual/Front_left_wheel/Front_left_roller_link2.STL" />
+                </geometry>
+                <material name="grey" />
+            </visual>
+            <collision>
+                <geometry>
+                    <mesh filename="package://omniman_description/meshes/visual/Front_left_wheel/Front_left_roller_link2.STL" />
+                </geometry>
+            </collision>
+            <inertial>
+                <mass value="0.009948" />
+                <origin xyz="0.000000 0.000000 0.000000" rpy="0 0 0" />
+                <inertia ixx="0.000001" ixy="0.000000" ixz="0.000000"
+                        iyy="0.000002" iyz="0.000000"
+                        izz="0.000002" />
+            </inertial>
+        </link>
+        <joint name="Front_left_roller_continuous_joint2" type="fixed">
+            <parent link="Front_left_plate_link" />
+            <child link="Front_left_roller_link2" />
+            <origin xyz="0.0184027 0.0259619 0.0340368" rpy="-0.0755575 0.342615 0.849182" />
+            <axis xyz="1 0 0" />
+        </joint>
+        <link name="Front_left_roller_link3">
+            <visual>
+                <geometry>
+                    <mesh filename="package://omniman_description/meshes/visual/Front_left_wheel/Front_left_roller_link3.STL" />
+                </geometry>
+                <material name="grey" />
+            </visual>
+            <collision>
+                <geometry>
+                    <mesh filename="package://omniman_description/meshes/visual/Front_left_wheel/Front_left_roller_link3.STL" />
+                </geometry>
+            </collision>
+            <inertial>
+                <mass value="0.009948" />
+                <origin xyz="0.000000 0.000000 0.000000" rpy="0 0 0" />
+                <inertia ixx="0.000001" ixy="0.000000" ixz="0.000000"
+                        iyy="0.000002" iyz="0.000000"
+                        izz="0.000002" />
+            </inertial>
+        </link>
+        <joint name="Front_left_roller_continuous_joint3" type="fixed">
+            <parent link="Front_left_plate_link" />
+            <child link="Front_left_roller_link3" />
+            <origin xyz="0.0359757 0.0259619 0.0142447" rpy="-0.88859 0.717228 1.21759" />
+            <axis xyz="1 0 0" />
+        </joint>
+        <link name="Front_left_roller_link4">
+            <visual>
+                <geometry>
+                    <mesh filename="package://omniman_description/meshes/visual/Front_left_wheel/Front_left_roller_link4.STL" />
+                </geometry>
+                <material name="grey" />
+            </visual>
+            <collision>
+                <geometry>
+                    <mesh filename="package://omniman_description/meshes/visual/Front_left_wheel/Front_left_roller_link4.STL" />
+                </geometry>
+            </collision>
+            <inertial>
+                <mass value="0.009948" />
+                <origin xyz="0.000000 0.000000 0.000000" rpy="0 0 0" />
+                <inertia ixx="0.000001" ixy="0.000000" ixz="0.000000"
+                        iyy="0.000002" iyz="0.000000"
+                        izz="0.000002" />
+            </inertial>
+        </link>
+        <joint name="Front_left_roller_continuous_joint4" type="fixed">
+            <parent link="Front_left_plate_link" />
+            <child link="Front_left_roller_link4" />
+            <origin xyz="0.0367153 0.0259619 -0.0122127" rpy="1.56019 0.735675 1.87604" />
+            <axis xyz="1 0 0" />
+        </joint>
+        <link name="Front_left_roller_link5">
+            <visual>
+                <geometry>
+                    <mesh filename="package://omniman_description/meshes/visual/Front_left_wheel/Front_left_roller_link5.STL" />
+                </geometry>
+                <material name="grey" />
+            </visual>
+            <collision>
+                <geometry>
+                    <mesh filename="package://omniman_description/meshes/visual/Front_left_wheel/Front_left_roller_link5.STL" />
+                </geometry>
+            </collision>
+            <inertial>
+                <mass value="0.009948" />
+                <origin xyz="0.000000 0.000000 0.000000" rpy="0 0 0" />
+                <inertia ixx="0.000001" ixy="0.000000" ixz="0.000000"
+                        iyy="0.000002" iyz="0.000000"
+                        izz="0.000002" />
+            </inertial>
+        </link>
+        <joint name="Front_left_roller_continuous_joint5" type="fixed">
+            <parent link="Front_left_plate_link" />
+            <child link="Front_left_roller_link5" />
+            <origin xyz="0.0202754 0.0259619 -0.0329556" rpy="0.652229 0.379944 2.27611" />
+            <axis xyz="1 0 0" />
+        </joint>
+        <link name="Front_left_roller_link6">
+            <visual>
+                <geometry>
+                    <mesh filename="package://omniman_description/meshes/visual/Front_left_wheel/Front_left_roller_link6.STL" />
+                </geometry>
+                <material name="grey" />
+            </visual>
+            <collision>
+                <geometry>
+                    <mesh filename="package://omniman_description/meshes/visual/Front_left_wheel/Front_left_roller_link6.STL" />
+                </geometry>
+            </collision>
+            <inertial>
+                <mass value="0.009948" />
+                <origin xyz="0.000000 0.000000 0.000000" rpy="0 0 0" />
+                <inertia ixx="0.000001" ixy="0.000000" ixz="0.000000"
+                        iyy="0.000002" iyz="0.000000"
+                        izz="0.000002" />
+            </inertial>
+        </link>
+        <joint name="Front_left_roller_continuous_joint6" type="fixed">
+            <parent link="Front_left_plate_link" />
+            <child link="Front_left_roller_link6" />
+            <origin xyz="-0.00565156 0.0259619 -0.0382783" rpy="-0.253974 -0.103067 2.35085" />
+            <axis xyz="1 0 0" />
+        </joint>
+        <link name="Front_left_roller_link7">
+            <visual>
+                <geometry>
+                    <mesh filename="package://omniman_description/meshes/visual/Front_left_wheel/Front_left_roller_link7.STL" />
+                </geometry>
+                <material name="grey" />
+            </visual>
+            <collision>
+                <geometry>
+                    <mesh filename="package://omniman_description/meshes/visual/Front_left_wheel/Front_left_roller_link7.STL" />
+                </geometry>
+            </collision>
+            <inertial>
+                <mass value="0.009948" />
+                <origin xyz="0.000000 0.000000 0.000000" rpy="0 0 0" />
+                <inertia ixx="0.000001" ixy="0.000000" ixz="0.000000"
+                        iyy="0.000002" iyz="0.000000"
+                        izz="0.000002" />
+            </inertial>
+        </link>
+        <joint name="Front_left_roller_continuous_joint7" type="fixed">
+            <parent link="Front_left_plate_link" />
+            <child link="Front_left_roller_link7" />
+            <origin xyz="-0.0289341 0.0259619 -0.0256901" rpy="-0.593154 -0.556829 2.1572" />
+            <axis xyz="1 0 0" />
+        </joint>
+        <link name="Front_left_roller_link_8">
+            <visual>
+                <geometry>
+                    <mesh filename="package://omniman_description/meshes/visual/Front_left_wheel/Front_left_roller_link8.STL" />
+                </geometry>
+                <material name="grey" />
+            </visual>
+            <collision>
+                <geometry>
+                    <mesh filename="package://omniman_description/meshes/visual/Front_left_wheel/Front_left_roller_link8.STL" />
+                </geometry>
+            </collision>
+            <inertial>
+                <mass value="0.009948" />
+                <origin xyz="0.000000 0.000000 0.000000" rpy="0 0 0" />
+                <inertia ixx="0.000001" ixy="0.000000" ixz="0.000000"
+                        iyy="0.000002" iyz="0.000000"
+                        izz="0.000002" />
+            </inertial>
+        </link>
+        <joint name="Front_left_roller_continuous_joint8" type="fixed">
+            <parent link="Front_left_plate_link" />
+            <child link="Front_left_roller_link_8" />
+            <origin xyz="-0.0386781 0.0259619 -0.00108124" rpy="-0.745113 -0.784992 1.5993" />
+            <axis xyz="1 0 0" />
+        </joint>
+        <link name="Front_left_roller_link_9">
+            <visual>
+                <geometry>
+                    <mesh filename="package://omniman_description/meshes/visual/Front_left_wheel/Front_left_roller_link9.STL" />
+                </geometry>
+                <material name="grey" />
+            </visual>
+            <collision>
+                <geometry>
+                    <mesh filename="package://omniman_description/meshes/visual/Front_left_wheel/Front_left_roller_link9.STL" />
+                </geometry>
+            </collision>
+            <inertial>
+                <mass value="0.009948" />
+                <origin xyz="0.000000 0.000000 0.000000" rpy="0 0 0" />
+                <inertia ixx="0.000001" ixy="0.000000" ixz="0.000000"
+                        iyy="0.000002" iyz="0.000000"
+                        izz="0.000002" />
+            </inertial>
+        </link>
+        <joint name="Front_left_roller_continuous_joint9" type="fixed">
+            <parent link="Front_left_plate_link" />
+            <child link="Front_left_roller_link_9" />
+            <origin xyz="-0.0303242 0.0259619 0.0240335" rpy="-0.366861 -0.587658 1.0153" />
+            <axis xyz="1 0 0" />
+        </joint>
         <!-- ==================== Rear_left Wheel ==================== -->
         <joint name="Rear_left_couple_fixed_joint" type="fixed">
@@ -109,4 +369,264 @@
             </inertial>
         </link>
+        <link name="Rear_left_plate_link">
+            <visual>
+                <geometry>
+                    <mesh filename="package://omniman_description/meshes/visual/Rear_left_wheel/Rear_left_plate_link.STL" />
+                </geometry>
+                <material name="grey" />
+            </visual>
+            <collision>
+                <geometry>
+                    <mesh filename="package://omniman_description/meshes/visual/Rear_left_wheel/Rear_left_plate_link.STL" />
+                </geometry>
+            </collision>
+            <inertial>
+                <mass value="0.330915" />
+                <origin xyz="-0.000002 0.025958 -0.000002" rpy="0 0 0" />
+                <inertia ixx="0.000188" ixy="0.000000" ixz="0.000000"
+                        iyy="0.000187" iyz="0.000000"
+                        izz="0.000188" />
+            </inertial>
+        </link>
+        <joint name="Rear_left_plate_continuous_joint" type="continuous">
+            <parent link="Rear_left_couple_link" />
+            <child link="Rear_left_plate_link" />
+            <origin xyz="0 0.01729 0" rpy="0 0 0" />
+            <axis xyz="0 1 0" />
+        </joint>
+        <link name="Rear_left_roller_link1">
+            <visual>
+                <geometry>
+                    <mesh filename="package://omniman_description/meshes/visual/Rear_left_wheel/Rear_left_roller_link1.STL" />
+                </geometry>
+                <material name="grey" />
+            </visual>
+            <collision>
+                <geometry>
+                    <mesh filename="package://omniman_description/meshes/visual/Rear_left_wheel/Rear_left_roller_link1.STL" />
+                </geometry>
+            </collision>
+            <inertial>
+                <mass value="0.009948" />
+                <origin xyz="0.000000 0.000000 0.000000" rpy="0 0 0" />
+                <inertia ixx="0.000001" ixy="0.000000" ixz="0.000000"
+                        iyy="0.000002" iyz="0.000000"
+                        izz="0.000002" />
+            </inertial>
+        </link>
+        <joint name="Rear_left_roller_continuous_joint1" type="fixed">
+            <parent link="Rear_left_plate_link" />
+            <child link="Rear_left_roller_link1" />
+            <origin xyz="-0.0056516 0.025962 0.038278" rpy="-0.057514 0.10307 2.3508" />
+            <axis xyz="-1 0 0" />
+        </joint>
+        <link name="Rear_left_roller_link2">
+            <visual>
+                <geometry>
+                    <mesh filename="package://omniman_description/meshes/visual/Rear_left_wheel/Rear_left_roller_link2.STL" />
+                </geometry>
+                <material name="grey" />
+            </visual>
+            <collision>
+                <geometry>
+                    <mesh filename="package://omniman_description/meshes/visual/Rear_left_wheel/Rear_left_roller_link2.STL" />
+                </geometry>
+            </collision>
+            <inertial>
+                <mass value="0.009948" />
+                <origin xyz="0.000000 0.000000 0.000000" rpy="0 0 0" />
+                <inertia ixx="0.000001" ixy="0.000000" ixz="0.000000"
+                        iyy="0.000002" iyz="0.000000"
+                        izz="0.000002" />
+            </inertial>
+        </link>
+        <joint name="Rear_left_roller_continuous_joint2" type="fixed">
+            <parent link="Rear_left_plate_link" />
+            <child link="Rear_left_roller_link2" />
+            <origin xyz="0.020275 0.025962 0.032956" rpy="0.44031 0.37994 -0.86548" />
+            <axis xyz="-1 0 0" />
+        </joint>
+        <link name="Rear_left_roller_link3">
+            <visual>
+                <geometry>
+                    <mesh filename="package://omniman_description/meshes/visual/Rear_left_wheel/Rear_left_roller_link3.STL" />
+                </geometry>
+                <material name="grey" />
+            </visual>
+            <collision>
+                <geometry>
+                    <mesh filename="package://omniman_description/meshes/visual/Rear_left_wheel/Rear_left_roller_link3.STL" />
+                </geometry>
+            </collision>
+            <inertial>
+                <mass value="0.009948" />
+                <origin xyz="0.000000 0.000000 0.000000" rpy="0 0 0" />
+                <inertia ixx="0.000001" ixy="0.000000" ixz="0.000000"
+                        iyy="0.000002" iyz="0.000000"
+                        izz="0.000002" />
+            </inertial>
+        </link>
+        <joint name="Rear_left_roller_continuous_joint3" type="fixed">
+            <parent link="Rear_left_plate_link" />
+            <child link="Rear_left_roller_link3" />
+            <origin xyz="0.036715 0.025962 0.012213" rpy="0.42911 0.73568 -1.2656" />
+            <axis xyz="-1 0 0" />
+        </joint>
+        <link name="Rear_left_roller_link4">
+            <visual>
+                <geometry>
+                    <mesh filename="package://omniman_description/meshes/visual/Rear_left_wheel/Rear_left_roller_link4.STL" />
+                </geometry>
+                <material name="grey" />
+            </visual>
+            <collision>
+                <geometry>
+                    <mesh filename="package://omniman_description/meshes/visual/Rear_left_wheel/Rear_left_roller_link4.STL" />
+                </geometry>
+            </collision>
+            <inertial>
+                <mass value="0.009948" />
+                <origin xyz="0.000000 0.000000 0.000000" rpy="0 0 0" />
+                <inertia ixx="0.000001" ixy="0.000000" ixz="0.000000"
+                        iyy="0.000002" iyz="0.000000"
+                        izz="0.000002" />
+            </inertial>
+        </link>
+        <joint name="Rear_left_roller_continuous_joint4" type="fixed">
+            <parent link="Rear_left_plate_link" />
+            <child link="Rear_left_roller_link4" />
+            <origin xyz="0.035976 0.025962 -0.014245" rpy="0.21486 0.71723 -1.924" />
+            <axis xyz="-1 0 0" />
+        </joint>
+        <link name="Rear_left_roller_link5">
+            <visual>
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