Commit message: Update enable base drive for omniman_vla immitation learning project, the goal are let the robot capable of doing base drive with nav2 while the arm maintain pick and place with immitation learning

File: omniman_vla/description/nxp_omniman.urdf.xacro (robot description, xacro)
@@ -2,5 +2,5 @@
 <robot name="nxp_omniman" xmlns:xacro="http://www.ros.org/wiki/xacro">
     <!-- Include the combined static URDF (base + arm) -->
-    <xacro:include filename="$(find omniman_vla)/urdf/omniman.urdf.xacro"/>
+     <xacro:include filename="$(find omniman_vla)/urdf/omniman.urdf.xacro"/>
     <!-- Include ros2_control hardware macros -->
     <xacro:include filename="$(find cybergear_control)/description/ros2_control/robstride.ros2_control.urdf.xacro"/>
@@ -8,7 +8,43 @@
     <!-- Launch arguments -->
     <xacro:property name="canbus_arm" default="can_arm"/>
+    <xacro:property name="canbus_base" default="can_base"/>
     <xacro:property name="serial_port" default="/dev/dynamixel"/>
     <!-- Instantiate the robot links/joints before adding ros2_control macros. -->
     <xacro:nxp_omniman/>
+    <!-- ========== Mecanum Wheels (CyberGear on canbus_base) ========== -->
+    <xacro:macro name="mecanum_wheel_ros2_control" params="name canbus device_id axis_direction joint_name">
+        <ros2_control name="${name}" type="actuator">
+            <hardware>
+                <plugin>cybergear_control/CybergearActuator</plugin>
+                <param name="can_interface">${canbus}</param>
+                <param name="timeout_sec">3.0</param>
+                <param name="interval_sec">0.01</param>
+                <param name="device_id">${device_id}</param>
+                <param name="primary_id">0</param>
+                <param name="effort_kp">500</param>
+                <param name="effort_kd">5</param>
+                <param name="axis_direction">${axis_direction}</param>
+            </hardware>
+            <joint name="${joint_name}">
+                <command_interface name="velocity"/>
+                <state_interface name="position"/>
+                <state_interface name="velocity"/>
+                <state_interface name="torque"/>
+                <state_interface name="temperature"/>
+            </joint>
+        </ros2_control>
+    </xacro:macro>
+    <xacro:mecanum_wheel_ros2_control
+        name="FrontLeftWheel" canbus="${canbus_base}"
+        device_id="3" axis_direction="-1" joint_name="Front_left_plate_continuous_joint"/>
+    <xacro:mecanum_wheel_ros2_control
+        name="FrontRightWheel" canbus="${canbus_base}"
+        device_id="4" axis_direction="1" joint_name="Front_right_plate_continuous_joint"/>
+    <xacro:mecanum_wheel_ros2_control
+        name="RearLeftWheel" canbus="${canbus_base}"
+        device_id="1" axis_direction="-1" joint_name="Rear_left_plate_continuous_joint"/>
+    <xacro:mecanum_wheel_ros2_control
+        name="RearRightWheel" canbus="${canbus_base}"
+        device_id="2" axis_direction="1" joint_name="Rear_right_plate_continuous_joint"/>
     <!-- ========== Arm Joints (CyberGear on canbus_arm) ========== -->
     <xacro:robstride_ros2_control name="ShoulderYaw" canbus="${canbus_arm}" device_id="5" joint_name="shoulder_yaw_joint" axis_direction="1"/>
