Commit message: Update Both xacros expand cleanly and their joint-name sets are now identical. I also parsed the SRDF against the generated URDF: no SRDF joint or link is missing from the model, and no actuated joint is missing from the SRDF. Your install space is --symlink-install, so all of these are already live — no rebuild needed for the teleop side.
Two things to know:
omniman_description/urdf/omniman_isaac.urdf still says left_finger_prismatic_joint. I left it deliberately — it pairs with omniman.usd, and if the USD carries its own joint names,
renaming only the URDF would desync the Isaac asset. Say the word if you want it aligned. The controller side is consistent now,
but I couldn't exercise the actual teleop run. When you launch it, the "complete state not yet known" warnings should stop immediately rather than repeating each second.

File: moveit_config/config/nxp_omniman.ros2_control.xacro (robot description, xacro)
@@ -50,8 +50,8 @@
                 <state_interface name="velocity"/>
             </joint>
-            <joint name="left_finger_prismatic_joint">
+            <joint name="gripper_prismatic_joint">
                 <command_interface name="position"/>
                 <state_interface name="position">
-                  <param name="initial_value">${initial_positions['left_finger_prismatic_joint']}</param>
+                  <param name="initial_value">${initial_positions['gripper_prismatic_joint']}</param>
                 </state_interface>
                 <state_interface name="velocity"/>

File: omniman_description/urdf/omniman.urdf (robot description, URDF)
Before this commit: robot nxp_omniman, 58 links, 57 joints
Joints:
- removed joint left_finger_prismatic_joint
- added joint gripper_prismatic_joint: type prismatic, parent palm_link, child left_finger_link, origin xyz=-0.016 -0.040 0.038 rpy=0 0 0, axis 0 -1 0, limit lower=-0.010 upper=0.019 effort=1 velocity=4.8
- joint right_finger_prismatic_joint: mimic joint=left_finger_prismatic_joint multiplier=-1.0 offset=0.0 -> joint=gripper_prismatic_joint multiplier=-1.0 offset=0.0

File: omniman_description/urdf/omniman.urdf.xacro (robot description, xacro)
@@ -1401,5 +1401,5 @@
         </joint>
         <link name="camera_optical_frame" />
-        <joint name="left_finger_prismatic_joint" type="prismatic">
+        <joint name="gripper_prismatic_joint" type="prismatic">
             <parent link="palm_link" />
             <child link="left_finger_link" />
@@ -1409,5 +1409,5 @@
         </joint>
         <joint name="right_finger_prismatic_joint" type="prismatic">
-            <mimic joint="left_finger_prismatic_joint" multiplier="-1.0" offset="0.0" />
+            <mimic joint="gripper_prismatic_joint" multiplier="-1.0" offset="0.0" />
             <parent link="palm_link" />
             <child link="right_finger_link" />

File: omniman_ros2_control/description/nxp_omniman.urdf.xacro (robot description, xacro)
@@ -81,5 +81,5 @@
                 <state_interface name="velocity"/>
             </joint>
-            <joint name="left_finger_prismatic_joint">
+            <joint name="gripper_prismatic_joint">
                 <command_interface name="position"/>
                 <state_interface name="position"/>
@@ -139,5 +139,5 @@
                                       />
         <xacro:dynamixel_ros2_control name="LeftFingerPrismatic" serial_device="${serial_port}" device_id="11"
-                                      joint_name="left_finger_prismatic_joint"
+                                      joint_name="gripper_prismatic_joint"
                                       use_prismatic="1"
                                       revolute_max="0.0" revolute_min="-2.5"
